File: uUSBHub.sch (KiCad schematic (older format))
At the start: 17 parts

Commit message: Add indicator LEDs
Parts:
- added D?: PORT 1, symbol Device:LED_Small
- added D?: PORT 2, symbol Device:LED_Small
- added D?: PORT 3, symbol Device:LED_Small
- added D?: PORT 4, symbol Device:LED_Small
- added D?: ACT/SUS, symbol Device:LED_Small
- added R? (x3): 1k, symbol Device:R_Small
Connections:
- net GND: now also R?.2
- net DRV: now reaches U?.22 (DRV)
- net DRV: now also D?.1 (K), D?.1 (K), D?.2 (A), D?.2 (A), D?.2 (A)
- net LED1: now reaches U?.23 (LED1/EESCL)
- net LED1: now also R?.1
- net LED2: now reaches U?.24 (LED2)
- net LED2: now also R?.1
- new net: D?.1 (K), D?.2 (A), R?.2 (x2)
- new net: D?.1 (K), R?.1
Changed lines of the file:
@@
 DUm
 Connection ~ 5750 1400
+$Comp
+L Device:LED_Small D?
+U 1 1 5F79372E
+P 9900 5150
+F 0 "D?" V 9946 5080 50  0000 R CNN
+F 1 "PORT 4" V 9855 5080 50  0000 R CNN
+F 2 "" V 9900 5150 50  0001 C CNN
+F 3 "~" V 9900 5150 50  0001 C CNN
+	1    9900 5150
+	0    -1   -1   0
+$EndComp
+$Comp
+L Device:LED_Small D?
+U 1 1 5F789F88
+P 9400 5150
+F 0 "D?" V 9354 5080 50  0000 R CNN
+F 1 "PORT 2" V 9445 5080 50  0000 R CNN
+F 2 "" V 9400 5150 50  0001 C CNN
+F 3 "~" V 9400 5150 50  0001 C CNN
+	1    9400 5150
+	0    -1   1    0
+$EndComp
+$Comp
+L Device:LED_Small D?
+U 1 1 5F78EDC8
+P 8950 5150
+F 0 "D?" V 8996 5080 50  0000 R CNN
+F 1 "PORT 3" V 8905 5080 50  0000 R CNN
+F 2 "" V 8950 5150 50  0001 C CNN
+F 3 "~" V 8950 5150 50  0001 C CNN
+	1    8950 5150
+	0    -1   -1   0
+$EndComp
+$Comp
+L Device:LED_Small D?
+U 1 1 5F788712
+P 8450 5150
+F 0 "D?" V 8404 5080 50  0000 R CNN
+F 1 "PORT 1" V 8495 5080 50  0000 R CNN
+F 2 "" V 8450 5150 50  0001 C CNN
+F 3 "~" V 8450 5150 50  0001 C CNN
+	1    8450 5150
+	0    -1   1    0
+$EndComp
+$Comp
+L Device:R_Small R?
+U 1 1 5F7B6CC9
+P 8700 4950
+F 0 "R?" H 8759 4996 50  0000 L CNN
+F 1 "1k" H 8759 4905 50  0000 L CNN
+F 2 "" H 8700 4950 50  0001 C CNN
+F 3 "~" H 8700 4950 50  0001 C CNN
+	1    8700 4950
+	1    0    0    -1
+$EndComp
+$Comp
+L Device:R_Small R?
+U 1 1 5F7B7805
+P 9650 4950
+F 0 "R?" H 9709 4996 50  0000 L CNN
+F 1 "1k" H 9709 4905 50  0000 L CNN
+F 2 "" H 9650 4950 50  0001 C CNN
+F 3 "~" H 9650 4950 50  0001 C CNN
+	1    9650 4950
+	1    0    0    -1
+$EndComp
+Text Label 8700 4750 1    50   ~ 0
+LED1
+Text Label 9650 4750 1    50   ~ 0
+LED2
+Text Label 9200 5450 3    50   ~ 0
+DRV
+Wire Wire Line
+	8700 4750 8700 4850
+Wire Wire Line
+	8450 5050 8700 5050
+Connection ~ 8700 5050
+Wire Wire Line
+	8700 5050 8950 5050
+Wire Wire Line
+	8450 5250 8700 5250
+Wire Wire Line
+	9400 5250 9650 5250
+Wire Wire Line
+	9900 5050 9650 5050
+Connection ~ 9650 5050
+Wire Wire Line
+	9650 5050 9400 5050
+Wire Wire Line
+	9650 4750 9650 4850
+Wire Wire Line
+	9650 5250 9650 5350
+Wire Wire Line
+	9650 5350 9200 5350
+Wire Wire Line
+	9200 5350 9200 5450
+Connection ~ 9650 5250
+Wire Wire Line
+	9650 5250 9900 5250
+Wire Wire Line
+	8700 5250 8700 5350
+Wire Wire Line
+	8700 5350 9200 5350
+Connection ~ 8700 5250
+Wire Wire Line
+	8700 5250 8950 5250
+Connection ~ 9200 5350
+Text Label 3200 3750 0    50   ~ 0
+LED1
+Text Label 3200 3850 0    50   ~ 0
+LED2
+Text Label 3200 3950 0    50   ~ 0
+DRV
+$Comp
+L Device:LED_Small D?
+U 1 1 5F7E0A1F
+P 10450 5150
+F 0 "D?" V 10496 5080 50  0000 R CNN
+F 1 "ACT/SUS" V 10405 5080 50  0000 R CNN
+F 2 "" V 10450 5150 50  0001 C CNN
+F 3 "~" V 10450 5150 50  0001 C CNN
+	1    10450 5150
+	0    -1   -1   0
+$EndComp
+$Comp
+L Device:R_Small R?
+U 1 1 5F7E1B19
+P 10450 5350
+F 0 "R?" H 10509 5396 50  0000 L CNN
+F 1 "1k" H 10509 5305 50  0000 L CNN
+F 2 "" H 10450 5350 50  0001 C CNN
+F 3 "~" H 10450 5350 50  0001 C CNN
+	1    10450 5350
+	1    0    0    -1
+$EndComp
+Text Label 10450 5000 1    50   ~ 0
+DRV
+Wire Wire Line
+	10450 5000 10450 5050
+$Comp
+L power:GND #PWR?
+U 1 1 5F7E8F2C
+P 10450 5450
+F 0 "#PWR?" H 10450 5200 50  0001 C CNN
+F 1 "GND" H 10455 5277 50  0000 C CNN
+F 2 "" H 10450 5450 50  0001 C CNN
+F 3 "" H 10450 5450 50  0001 C CNN
+	1    10450 5450
+	1    0    0    -1
+$EndComp
 $EndSCHEMATC

Commit message: Mopping up remaining IC control pins
Parts:
- added R?: 2k7 1%, symbol Device:R_Small
- added Y?: 12MHz, symbol Device:Crystal_Small
Connections:
- net GND: now also U?.19 (BUSJ), R?.2
- net VBUS: now also U?.18 (VBUSM), U?.20 (VDD5)
- net +1V8: now reaches C?.1, U?.12 (VD18_O), U?.28 (VD18)
- net +3V3: now reaches C?.1, U?.13 (VD33), U?.21 (VD33_O)
- net +3V3: now also U?.17 (~XRSTJ), U?.26 (OVCJ)
- net at U?.14 (REXT): now also R?.1
- net at U?.2 (XOUT): now also Y?.2
- net at U?.3 (XIN): now also Y?.1
- no-connect marks 5 -> 7
Changed lines of the file:
@@
 	1    0    0    -1
 $EndComp
+NoConn ~ 3200 3650
+$Comp
+L power:GND #PWR?
+U 1 1 5F8014E0
+P 1500 3000
+F 0 "#PWR?" H 1500 2750 50  0001 C CNN
+F 1 "GND" H 1505 2827 50  0000 C CNN
+F 2 "" H 1500 3000 50  0001 C CNN
+F 3 "" H 1500 3000 50  0001 C CNN
+	1    1500 3000
+	1    0    0    -1
+$EndComp
+Wire Wire Line
+	1800 2950 1500 2950
+Wire Wire Line
+	1500 2950 1500 3000
+$Comp
+L power:+3V3 #PWR?
+U 1 1 5F805F29
+P 2500 1700
+F 0 "#PWR?" H 2500 1550 50  0001 C CNN
+F 1 "+3V3" H 2515 1873 50  0000 C CNN
+F 2 "" H 2500 1700 50  0001 C CNN
+F 3 "" H 2500 1700 50  0001 C CNN
+	1    2500 1700
+	1    0    0    -1
+$EndComp
+Connection ~ 2500 1700
+$Comp
+L power:+1V8 #PWR?
+U 1 1 5F8070E8
+P 2850 1700
+F 0 "#PWR?" H 2850 1550 50  0001 C CNN
+F 1 "+1V8" H 2865 1873 50  0000 C CNN
+F 2 "" H 2850 1700 50  0001 C CNN
+F 3 "" H 2850 1700 50  0001 C CNN
+	1    2850 1700
+	1    0    0    -1
+$EndComp
+Connection ~ 2850 1700
+Wire Wire Line
+	1800 3050 1600 3050
+Wire Wire Line
+	1600 3050 1600 2850
+Wire Wire Line
+	1600 2850 1800 2850
+$Comp
+L power:+3V3 #PWR?
+U 1 1 5F80B9F0
+P 1500 2850
+F 0 "#PWR?" H 1500 2700 50  0001 C CNN
+F 1 "+3V3" H 1515 3023 50  0000 C CNN
+F 2 "" H 1500 2850 50  0001 C CNN
+F 3 "" H 1500 2850 50  0001 C CNN
+	1    1500 2850
+	1    0    0    -1
+$EndComp
+Wire Wire Line
+	1600 2850 1500 2850
+Connection ~ 1600 2850
+$Comp
+L Device:R_Small R?
+U 1 1 5F8107B3
+P 1800 4250
+F 0 "R?" H 1650 4300 50  0000 L CNN
+F 1 "2k7 1%" H 1450 4200 50  0000 L CNN
+F 2 "" H 1800 4250 50  0001 C CNN
+F 3 "~" H 1800 4250 50  0001 C CNN
+	1    1800 4250
+	1    0    0    -1
+$EndComp
+$Comp
+L power:GND #PWR?
+U 1 1 5F8122E4
+P 1800 4350
+F 0 "#PWR?" H 1800 4100 50  0001 C CNN
+F 1 "GND" H 1805 4177 50  0000 C CNN
+F 2 "" H 1800 4350 50  0001 C CNN
+F 3 "" H 1800 4350 50  0001 C CNN
+	1    1800 4350
+	1    0    0    -1
+$EndComp
+NoConn ~ 3200 4150
+$Comp
+L power:VBUS #PWR?
+U 1 1 5F816207
+P 1800 2150
+F 0 "#PWR?" H 1800 2000 50  0001 C CNN
+F 1 "VBUS" H 1815 2323 50  0000 C CNN
+F 2 "" H 1800 2150 50  0001 C CNN
+F 3 "" H 1800 2150 50  0001 C CNN
+	1    1800 2150
+	1    0    0    -1
+$EndComp
+Wire Wire Line
+	2300 2150 1800 2150
+Wire Wire Line
+	1800 2150 1800 2350
+Connection ~ 1800 2150
+$Comp
+L Device:Crystal_Small Y?
+U 1 1 5F821341
+P 1150 3900
+F 0 "Y?" V 1200 4100 50  0000 R CNN
+F 1 "12MHz" V 1100 4250 50  0000 R CNN
+F 2 "" H 1150 3900 50  0001 C CNN
+F 3 "~" H 1150 3900 50  0001 C CNN
+	1    1150 3900
+	0    -1   -1   0
+$EndComp
+Wire Wire Line
+	1800 3950 1250 3950
+Wire Wire Line
+	1250 3950 1250 4000
+Wire Wire Line
+	1250 4000 1150 4000
+Wire Wire Line
+	1800 3850 1250 3850
+Wire Wire Line
+	1250 3850 1250 3800
+Wire Wire Line
+	1250 3800 1150 3800
 $EndSCHEMATC

Commit message: Correct some extra pins bits, also add 5v decoupling
Parts:
- added C?: 10u, symbol Device:C_Small
- added C?: 4u7, symbol Device:C_Small
- added C?: 100n, symbol Device:C_Small
- added R?: 47k, symbol Device:R_Small
- added R? (x2): 100k, symbol Device:R_Small
- added R?: 10k, symbol Device:R_Small
Connections:
- net +3V3: no longer U?.17 (~XRSTJ)
- net GND: now also C?.2, C?.2, C?.2, R?.2, R?.2; no longer U?.19 (BUSJ)
- net VBUS: now also C?.1, C?.1, C?.1, R?.1, R?.1; no longer U?.18 (VBUSM)
- new net: R?.2, U?.17 (~XRSTJ)
- new net: R?.1, R?.2, U?.18 (VBUSM)
- new net: R?.1, U?.19 (BUSJ)
Other:
- moved on the sheet: C?, D?, R?, U?, Y?

Commit message: Initial footprint assignment for header version
Parts:
- C1, C2, C6, C7, C8, C9: renamed from C?; footprint (none) -> Capacitor_SMD:C_0603_1608Metric
- C3, C4, C5: renamed from C?; footprint (none) -> Capacitor_SMD:C_0805_2012Metric
- D1, D2, D3, D4, D5: renamed from D?; footprint (none) -> LED_SMD:LED_0805_2012Metric
- J1, J2, J3, J4, J5: renamed from J?; footprint (none) -> Connector_PinHeader_2.54mm:PinHeader_1x05_P2.54mm_Vertical
- R1, R2, R3, R4, R5, R6, R7, R8: renamed from R?; footprint (none) -> Resistor_SMD:R_0603_1608Metric
- gave numbers to parts that had none: 7

Commit message: Tweak the data line names to properly allow differential pair routing
Connections:
- net D1m renamed D1-
- net D1p renamed D1+
- net D2m renamed D2-
- net D2p renamed D2+
- net D3m renamed D3-
- net D3p renamed D3+
- net D4m renamed D4-
- net D4p renamed D4+
- net DUm renamed DU-
- net DUp renamed DU+
Changed lines of the file:
@@
 	6650 1400 6900 1400
 Text Label 7100 3150 3    50   ~ 0
-D1p
+D1+
 Text Label 7200 3150 3    50   ~ 0
-D1m
+D1-
 Wire Wire Line
 	7200 3050 7200 3150
@@
 	8250 3050 8250 3150
 Text Label 8250 3150 3    50   ~ 0
-D2p
+D2+
 Text Label 8350 3150 3    50   ~ 0
-D2m
+D2-
 Wire Wire Line
 	8350 3050 8350 3150
@@
 	9400 3050 9400 3150
 Text Label 9400 3150 3    50   ~ 0
-D3p
+D3+
 Text Label 9500 3150 3    50   ~ 0
-D3m
+D3-
 Wire Wire Line
 	9500 3050 9500 3150
@@
 	10550 3050 10550 3150
 Text Label 10550 3150 3    50   ~ 0
-D4p
+D4+
 Text Label 10650 3150 3    50   ~ 0
-D4m
+D4-
 Wire Wire Line
 	10650 3050 10650 3150
@@
 	5600 3050 5950 3050
 Text Label 3050 1550 0    50   ~ 0
-D1p
+D1+
 Text Label 3050 1650 0    50   ~ 0
-D1m
+D1-
 Text Label 3050 1850 0    50   ~ 0
-D2p
+D2+
 Text Label 3050 1950 0    50   ~ 0
-D2m
+D2-
 Text Label 3050 2150 0    50   ~ 0
-D3p
+D3+
 Text Label 3050 2250 0    50   ~ 0
-D3m
+D3-
 Text Label 3050 2450 0    50   ~ 0
-D4p
+D4+
 Text Label 3050 2550 0    50   ~ 0
-D4m
+D4-
 Wire Wire Line
 	2650 1350 2700 1350
@@
 	5500 1400 5750 1400
 Text Label 5950 3150 3    50   ~ 0
-DUp
+DU+
 Text Label 6050 3150 3    50   ~ 0
-DUm
+DU-
 Wire Wire Line
 	6050 3150 6050 3050
@@
 	5950 3150 5950 3050
 Text Label 1650 1750 2    50   ~ 0
-DUp
+DU+
 Text Label 1650 1850 2    50   ~ 0
-DUm
+DU-
 Connection ~ 5750 1400
 $Comp

Commit message: WIP
Parts:
- removed J1: UPSTREAM, Connector_PinHeader_2.54mm:PinHeader_1x05_P2.54mm_Vertical, symbol Connector:USB_A
- added H1, H2, H3, H4: MountingHole, MountingHole:MountingHole_3.2mm_M3_ISO14580, symbol Mechanical:MountingHole
- added J1: USB_B_Micro, uUSBHub:U254-051T-4BH83-F1S, symbol Connector:USB_B_Micro
- J2, J3, J4, J5: footprint Connector_PinHeader_2.54mm:PinHeader_1x05_P2.54mm_Vertical -> uUSBHub:JTJ-USB-AF-08
Connections:
- net D1+: now also U2.3 (I/O2); no longer U2.1 (I/O1)
- net D1-: now also U2.1 (I/O1); no longer U2.3 (I/O2)
- net D4+: now also U5.3 (I/O2); no longer U5.1 (I/O1)
- net D4-: now also U5.1 (I/O1); no longer U5.3 (I/O2)
- net GND: now also J1.5 (GND)
- net VBUS: now also J1.1 (VBUS)
- net at J2.2 (D-): now also U2.6 (I/O1); no longer U2.4 (I/O2)
- net at J2.3 (D+): now also U2.4 (I/O2); no longer U2.6 (I/O1)
- net at J5.2 (D-): now also U5.6 (I/O1); no longer U5.4 (I/O2)
- net at J5.3 (D+): now also U5.4 (I/O2); no longer U5.6 (I/O1)
- net at U1.4 (I/O2): now also J1.2 (D-)
- net at U1.6 (I/O1): now also J1.3 (D+)
- no-connect marks 7 -> 8
Changed lines of the file:
@@
 F 0 "J2" V 6733 993 50  0000 C CNN
 F 1 "PORT1" V 6824 993 50  0000 C CNN
-F 2 "Connector_PinHeader_2.54mm:PinHeader_1x05_P2.54mm_Vertical" H 7250 1000 50  0001 C CNN
+F 2 "uUSBHub:JTJ-USB-AF-08" H 7250 1000 50  0001 C CNN
 F 3 " ~" H 7250 1000 50  0001 C CNN
 	1    7100 1050
@@
 F 0 "J3" V 7883 993 50  0000 C CNN
 F 1 "PORT2" V 7974 993 50  0000 C CNN
-F 2 "Connector_PinHeader_2.54mm:PinHeader_1x05_P2.54mm_Vertical" H 8400 1000 50  0001 C CNN
+F 2 "uUSBHub:JTJ-USB-AF-08" H 8400 1000 50  0001 C CNN
 F 3 " ~" H 8400 1000 50  0001 C CNN
 	1    8250 1050
@@
 F 0 "J4" V 9033 993 50  0000 C CNN
 F 1 "PORT3" V 9124 993 50  0000 C CNN
-F 2 "Connector_PinHeader_2.54mm:PinHeader_1x05_P2.54mm_Vertical" H 9550 1000 50  0001 C CNN
+F 2 "uUSBHub:JTJ-USB-AF-08" H 9550 1000 50  0001 C CNN
 F 3 " ~" H 9550 1000 50  0001 C CNN
 	1    9400 1050
@@
 F 0 "J5" V 10183 993 50  0000 C CNN
 F 1 "PORT4" V 10274 993 50  0000 C CNN
-F 2 "Connector_PinHeader_2.54mm:PinHeader_1x05_P2.54mm_Vertical" H 10700 1000 50  0001 C CNN
+F 2 "uUSBHub:JTJ-USB-AF-08" H 10700 1000 50  0001 C CNN
 F 3 " ~" H 10700 1000 50  0001 C CNN
 	1    10550 1050
@@
 F 3 "https://www.st.com/resource/en/datasheet/usblc6-2.pdf" H 10800 2750 50  0001 C CNN
 	1    10600 2400
-	1    0    0    -1
+	-1   0    0    -1
 $EndComp
 Wire Wire Line
@@
 F 3 "https://www.st.com/resource/en/datasheet/usblc6-2.pdf" H 7350 2750 50  0001 C CNN
 	1    7150 2400
-	1    0    0    -1
+	-1   0    0    -1
 $EndComp
 Wire Wire Line
@@
 Wire Wire Line
 	10650 3050 10650 3150
-$Comp
-L Connector:USB_A J1
-U 1 1 5F752C62
-P 5950 1050
-F 0 "J1" V 5600 950 50  0000 L CNN
-F 1 "UPSTREAM" V 5700 900 50  0000 L CNN
-F 2 "Connector_PinHeader_2.54mm:PinHeader_1x05_P2.54mm_Vertical" H 6100 1000 50  0001 C CNN
-F 3 " ~" H 6100 1000 50  0001 C CNN
-	1    5950 1050
-	0    -1   1    0
-$EndComp
 NoConn ~ 6350 950
 $Comp
@@
 	0    1    1    0
 $EndComp
+$Comp
+L Connector:USB_B_Micro J1
+U 1 1 5F81299F
+P 5950 1050
+F 0 "J1" V 5583 993 50  0000 C CNN
+F 1 "USB_B_Micro" V 5674 993 50  0000 C CNN
+F 2 "uUSBHub:U254-051T-4BH83-F1S" H 6100 1000 50  0001 C CNN
+F 3 "~" H 6100 1000 50  0001 C CNN
+	1    5950 1050
+	0    -1   1    0
+$EndComp
 Connection ~ 6350 1050
+NoConn ~ 6150 1350
+$Comp
+L Mechanical:MountingHole H4
+U 1 1 5F850554
+P 6250 7600
+F 0 "H4" H 6350 7646 50  0000 L CNN
+F 1 "MountingHole" H 6350 7555 50  0000 L CNN
+F 2 "MountingHole:MountingHole_3.2mm_M3_ISO14580" H 6250 7600 50  0001 C CNN
+F 3 "~" H 6250 7600 50  0001 C CNN
+	1    6250 7600
+	1    0    0    -1
+$EndComp
+$Comp
+L Mechanical:MountingHole H3
+U 1 1 5F852139
+P 6250 7400
+F 0 "H3" H 6350 7446 50  0000 L CNN
+F 1 "MountingHole" H 6350 7355 50  0000 L CNN
+F 2 "MountingHole:MountingHole_3.2mm_M3_ISO14580" H 6250 7400 50  0001 C CNN
+F 3 "~" H 6250 7400 50  0001 C CNN
+	1    6250 7400
+	1    0    0    -1
+$EndComp
+$Comp
+L Mechanical:MountingHole H2
+U 1 1 5F8522C0
+P 6250 7200
+F 0 "H2" H 6350 7246 50  0000 L CNN
+F 1 "MountingHole" H 6350 7155 50  0000 L CNN
+F 2 "MountingHole:MountingHole_3.2mm_M3_ISO14580" H 6250 7200 50  0001 C CNN
+F 3 "~" H 6250 7200 50  0001 C CNN
+	1    6250 7200
+	1    0    0    -1
+$EndComp
+$Comp
+L Mechanical:MountingHole H1
+U 1 1 5F8524E3
+P 6250 7000
+F 0 "H1" H 6350 7046 50  0000 L CNN
+F 1 "MountingHole" H 6350 6955 50  0000 L CNN
+F 2 "MountingHole:MountingHole_3.2mm_M3_ISO14580" H 6250 7000 50  0001 C CNN
+F 3 "~" H 6250 7000 50  0001 C CNN
+	1    6250 7000
+	1    0    0    -1
+$EndComp
 $EndSCHEMATC
